File: PCB/Arduino101/board1.brd (EAGLE design)
At the start: 72.1 x 66 mm, 41 parts

Commit message: autorouted
Routing:
- net GND: track 0.00 -> 272.8 mm
- net 3V3: track 0.00 -> 106.5 mm
- net 14V8: track 0.00 -> 70.6 mm
- net N$5: track 0.00 -> 43.0 mm
- net BRAKE_PWM3: track 0.00 -> 27.0 mm
- net STEERING_P: track 0.00 -> 25.5 mm
- net WHEEL_P1: track 0.00 -> 23.0 mm
- net BRAKE_P1: track 0.00 -> 22.7 mm
- net WHEEL_P2: track 0.00 -> 21.6 mm
- net WHEEL_P3: track 0.00 -> 20.7 mm
- net BRAKE_P2: track 0.00 -> 20.3 mm
- net BRAKE_P3: track 0.00 -> 19.0 mm
- net TILT_P: track 0.00 -> 18.5 mm
- net BRAKE_PWM2: track 0.00 -> 17.4 mm
- net TILT_PWM: track 0.00 -> 17.1 mm
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